File: MTJ_chipholder.kicad_sch (KiCad schematic)
At the start: 5 parts, among them J1 8428-21B1-RK-TR

Commit message: v1.0
Parts:
- removed InputProbe1, OutputProbe1: TestPoint, Connector_PinSocket_2.54mm:PinSocket_1x01_P2.54mm_Vertical, symbol Connector:TestPoint
- added J2, J3: Conn_01x02_Pin, Connector_PinSocket_2.54mm:PinSocket_1x02_P2.54mm_Vertical, symbol Connector:Conn_01x02_Pin
Connections:
- net GND: now also J2.2 (Pin_2), J3.1 (Pin_1)
- net mtjin1: now also J3.2 (Pin_2)
- net mtjout1: now also J2.1 (Pin_1)
Other:
- moved on the sheet: SMA-out1
