File: MTJ_chipholder.kicad_pcb (KiCad board)
At the start: 4 copper layers, 74 x 35.5 mm, 5 parts, among them J1 8428-21B1-RK-TR

Commit message: v1.0
Parts:
- removed InputProbe1, OutputProbe1: TestPoint, Connector_PinSocket_2.54mm:PinSocket_1x01_P2.54mm_Vertical
- added J2: Conn_01x02_Pin, Connector_PinSocket_2.54mm:PinSocket_1x02_P2.54mm_Vertical, F.Cu at (132.2, 75.0)
- added J3: Conn_01x02_Pin, Connector_PinSocket_2.54mm:PinSocket_1x02_P2.54mm_Vertical, F.Cu at (89.1, 74.7)
Routing:
- net /mtjin1: track 25.0 -> 30.6 mm
- net /mtjout1: track 25.8 -> 30.4 mm
- net GND: vias 20 -> 36
- added copper zone on B.Cu, net GND
Other:
- board text added: "MTJ chip holder v1.0 Troy Criss and Andy Haas, NYU March 2026"

Commit message: v1.0 with biggerness gerbers
Parts:
- added REF**: MountingHole_2mm, MountingHole:MountingHole_2mm, F.Cu at (78.2, 73.6)
- added REF**: MountingHole_2mm, MountingHole:MountingHole_2mm, F.Cu at (78.2, 115.4)
- added REF**: MountingHole_2mm, MountingHole:MountingHole_2mm, F.Cu at (209.4, 73.4)
- added REF**: MountingHole_2mm, MountingHole:MountingHole_2mm, F.Cu at (208.8, 115.3)
- moved J1 10.4 mm to (109.7, 96.0)
- moved J2 10.4 mm to (131.7, 85.4)
- moved J3 10.4 mm to (88.7, 85.1)
- moved SMA-in1 10.4 mm to (88.2, 98.5)
- moved SMA-out1 10.4 mm to (131.9, 98.5)
Other:
- board size 74 x 35.5 mm -> 138.8 x 50.7 mm
